Commit message: 最后一步,视觉抓取

File: src/universal_robot/ur_description/urdf/ur5_robotiq85_gripper.urdf.xacro (robot description, xacro)
@@ -1,6 +1,9 @@
 <?xml version="1.0"?>
 <robot name="ur5" xmlns:xacro="http://www.ros.org/wiki/xacro">
+  <xacro:property name="M_PI" value="3.1415926536"/>
   <xacro:include filename="$(find ur_description)/urdf/ur5_joint_limited_robot.urdf.xacro" />
   <xacro:include filename="$(find robotiq_description)/urdf/robotiq_85_gripper.urdf.xacro" />
+  <xacro:include filename="$(find ur_description)/urdf/camera.urdf.xacro" />
+  <xacro:include filename="$(find ur_description)/urdf/materials.urdf.xacro" />
   <!-- Robotiq Coupler -->
   <!--  + Height added by the coupler: 8mm -->
