Commit message: vision and model

File: src/universal_robot/ur_description/urdf/camera.urdf.xacro (robot description, xacro)
@@ -5,5 +5,5 @@
 <robot name="camera" xmlns:xacro="http://ros.org/wiki/xacro">
    <joint name="camera_joint" type="fixed">
-        <origin xyz="0.5 0 1.2" rpy="0 ${M_PI/2} 0"/>
+        <origin xyz="0.7 0 1" rpy="0 ${M_PI/2} 0"/>
         <parent link="base_link"/>
         <child link="camera_link"/>

File: src/universal_robot/ur_description/urdf/ur5_robotiq85_gripper.urdf.xacro (robot description, xacro)
@@ -2,8 +2,8 @@
 <robot name="ur5" xmlns:xacro="http://www.ros.org/wiki/xacro">
   <xacro:property name="M_PI" value="3.1415926536"/>
+  <xacro:include filename="$(find ur_description)/urdf/materials.urdf.xacro" />
   <xacro:include filename="$(find ur_description)/urdf/ur5_joint_limited_robot.urdf.xacro" />
   <xacro:include filename="$(find robotiq_description)/urdf/robotiq_85_gripper.urdf.xacro" />
   <xacro:include filename="$(find ur_description)/urdf/camera.urdf.xacro" />
-  <xacro:include filename="$(find ur_description)/urdf/materials.urdf.xacro" />
   <!-- Robotiq Coupler -->
   <!--  + Height added by the coupler: 8mm -->
